Commit message: change

File: src/marscar_gazebo_ros2/urdf/marsrover_control.urdf.xacro (robot description, xacro)
@@ -29,4 +29,5 @@
   </joint>
   <joint name="left_foot1" type="revolute">
+    <dynamics damping="1" friction="1"/>
     <limit lower="-0.5000" upper="0.5000" effort="10000.00000" velocity="5.00000"/>
     <origin rpy="0.00000 0.00000 0.00000" xyz="0.22877 0.03703 -0.11721"/>
@@ -36,4 +37,5 @@
   </joint>
   <joint name="left_foot3" type="revolute">
+    <dynamics damping="1" friction="1"/>
     <limit lower="-0.5000" upper="0.5000" effort="10000.00000" velocity="5.00000"/>
     <origin rpy="0.00000 0.00000 0.00000" xyz="-0.14234 0.03054 -0.04748"/>
@@ -79,4 +81,5 @@
   </joint>
   <joint name="right_foot1" type="revolute">
+    <dynamics damping="1" friction="1"/>
     <limit lower="-0.5000" upper="0.5000" effort="10000.00000" velocity="5.00000"/>
     <origin rpy="0.00000 0.00000 0.00000" xyz="0.22441 -0.04260 -0.11148"/>
@@ -86,4 +89,5 @@
   </joint>
   <joint name="right_foot3" type="revolute">
+    <dynamics damping="1" friction="1"/>
     <limit lower="-0.5000" upper="0.5000" effort="10000.00000" velocity="5.00000"/>
     <origin rpy="0.00000 0.00000 0.00000" xyz="-0.13920 -0.03213 -0.04813"/>
@@ -420,5 +424,5 @@
     <color rgba="0.01961 0.00000 0.00000 1.00000"/>
   </material>
-  <ros2_control name="GazeboSystem" type="system">
+  <!-- <ros2_control name="GazeboSystem" type="system">
     <hardware>
       <plugin>gazebo_ros2_control/GazeboSystem</plugin>
@@ -578,5 +582,5 @@
       <parameters>$(find marscar_gazebo_ros2)/config/mars_car_controller.yaml</parameters>
     </plugin>
-  </gazebo>
+  </gazebo> -->
   <gazebo>
     <plugin name="odom_pub_plugin" filename="libgazebo_ros_odom.so">
@@ -602,4 +606,48 @@
       <topic>my_robot/ball_shooter/fire</topic>
     </plugin>
+     <plugin name="gazebo_ros_ackermann_drive" filename="libmarsrover_control.so">
+      <ros>
+        <namespace>demo</namespace>
+        <remapping>cmd_vel:=cmd_demo</remapping>
+        <remapping>odom:=odom_demo</remapping>
+        <remapping>distance:=distance_demo</remapping>
+        <remapping>steerangle:=steerangle_demo</remapping>
+      </ros>
+      <update_rate>100.0</update_rate>
+      <!-- wheels -->
+      <front_left_joint>left_wheel1</front_left_joint>
+      <front_right_joint>right_wheel1</front_right_joint>
+      <rear_left_joint>left_wheel3</rear_left_joint>
+      <rear_right_joint>right_wheel3</rear_right_joint>
+      <middle_left_joint>left_wheel2</middle_left_joint>
+      <middle_right_joint>right_wheel2</middle_right_joint>
+      <left_steering_joint>left_foot1</left_steering_joint>
+      <right_steering_joint>right_foot1</right_steering_joint>
+      <left_rear_steering_joint>left_foot3</left_rear_steering_joint>
+      <right_rear_steering_joint>right_foot3</right_rear_steering_joint>
+      <steering_wheel_joint>arm1</steering_wheel_joint>
+      <!-- Max absolute steer angle for tyre in radians-->
+      <!-- Any cmd_vel angular z greater than this would be capped -->
+      <max_steer>0.6458</max_steer>
+      <!-- Max absolute steering angle of steering wheel -->
+      <max_steering_angle>7.85</max_steering_angle>
+      <!-- Max absolute linear speed in m/s -->
+      <max_speed>2</max_speed>
+      <!-- PID tuning -->
+      <left_steering_pid_gain>500 10 5</left_steering_pid_gain>
+      <left_steering_i_range>-1000 1000</left_steering_i_range>
+      <right_steering_pid_gain>500 10 5</right_steering_pid_gain>
+      <right_steering_i_range>-1000 1000</right_steering_i_range>
+      <linear_velocity_pid_gain>500 10 5</linear_velocity_pid_gain>
+      <linear_velocity_i_range>-1000 1000</linear_velocity_i_range>
+      <!-- output -->
+      <publish_odom>false</publish_odom>
+      <publish_odom_tf>false</publish_odom_tf>
+      <publish_wheel_tf>false</publish_wheel_tf>
+      <publish_distance>false</publish_distance>
+      <publish_steerangle>false</publish_steerangle>
+      <odometry_frame>odom_demo</odometry_frame>
+      <robot_base_frame>base_link</robot_base_frame>
+    </plugin>
   </gazebo>
   <xacro:include filename="$(find marscar_gazebo_ros2)/sensor_description/inertial_macros.xacro" />
